File: CurrentSinkOrSwim/CurrentSinkOrSwim.sch (KiCad schematic (older format))
At the start: 0 parts

Commit message: Adding preliminary components (without values) to the schematic
Parts:
- added C? (x2): C, ~, symbol C
- added P?: CONN_2, symbol CONN_2
- added Q?: MOSFET_N, ~, symbol MOSFET_N
- added R? (x2): R, ~, symbol R
- added RV?: POT, ~, symbol POT
- added U? (x2): LMV358, symbol LMV358
- added U?: TC1016, ~, symbol TC1016
Connections:
- net labels added: GND
- wire segments 0 -> 36
Changed lines of the file:
@@
 LIBS:contrib
 LIBS:valves
+LIBS:CurrentSinkOrSwim.lib
+LIBS:CurrentSinkOrSwim-cache
 EELAYER 27 0
 EELAYER END
@@
 Comment4 ""
 $EndDescr
+$Comp
+L LMV358 U?
+U 1 1 55D776C3
+P 4700 3900
+F 0 "U?" H 4650 4100 60  0000 L CNN
+F 1 "LMV358" H 4650 3650 60  0000 L CNN
+F 2 "" H 4700 3900 60  0000 C CNN
+F 3 "" H 4700 3900 60  0000 C CNN
+	1    4700 3900
+	1    0    0    -1
+$EndComp
+$Comp
+L R R?
+U 1 1 55D776EA
+P 6050 5150
+F 0 "R?" V 6130 5150 40  0000 C CNN
+F 1 "R" V 6057 5151 40  0000 C CNN
+F 2 "~" V 5980 5150 30  0000 C CNN
+F 3 "~" H 6050 5150 30  0000 C CNN
+	1    6050 5150
+	1    0    0    -1
+$EndComp
+$Comp
+L GND #PWR?
+U 1 1 55D776FA
+P 6050 5850
+F 0 "#PWR?" H 6050 5850 30  0001 C CNN
+F 1 "GND" H 6050 5780 30  0001 C CNN
+F 2 "~" H 6050 5850 60  0000 C CNN
+F 3 "~" H 6050 5850 60  0000 C CNN
+	1    6050 5850
+	1    0    0    -1
+$EndComp
+$Comp
+L MOSFET_N Q?
+U 1 1 55D7770C
+P 5950 3900
+F 0 "Q?" H 5960 4070 60  0000 R CNN
+F 1 "MOSFET_N" H 5960 3750 60  0000 R CNN
+F 2 "~" H 5950 3900 60  0000 C CNN
+F 3 "~" H 5950 3900 60  0000 C CNN
+	1    5950 3900
+	1    0    0    -1
+$EndComp
+$Comp
+L R R?
+U 1 1 55D77732
+P 2350 5400
+F 0 "R?" V 2430 5400 40  0000 C CNN
+F 1 "R" V 2357 5401 40  0000 C CNN
+F 2 "~" V 2280 5400 30  0000 C CNN
+F 3 "~" H 2350 5400 30  0000 C CNN
+	1    2350 5400
+	1    0    0    -1
+$EndComp
+$Comp
+L GND #PWR?
+U 1 1 55D7776F
+P 4600 4450
+F 0 "#PWR?" H 4600 4450 30  0001 C CNN
+F 1 "GND" H 4600 4380 30  0001 C CNN
+F 2 "~" H 4600 4450 60  0000 C CNN
+F 3 "~" H 4600 4450 60  0000 C CNN
+	1    4600 4450
+	1    0    0    -1
+$EndComp
+Wire Wire Line
+	6050 5400 6050 5750
+Wire Wire Line
+	6050 5750 6050 5850
+Wire Wire Line
+	6050 4100 6050 4650
+Wire Wire Line
+	6050 4650 6050 4900
+Wire Wire Line
+	5200 3900 5750 3900
+Wire Wire Line
+	4600 4300 4600 4450
+Wire Wire Line
+	4600 2600 4600 3500
+Wire Wire Line
+	2650 2600 4600 2600
+Wire Wire Line
+	4600 2600 4800 2600
+Wire Wire Line
+	4800 2600 4900 2600
+Wire Wire Line
+	2350 4800 2350 4950
+Wire Wire Line
+	2350 4950 2350 5150
+Wire Wire Line
+	4200 4000 3950 4000
+Wire Wire Line
+	3950 4000 3950 4650
+Wire Wire Line
+	3950 4650 6050 4650
+Connection ~ 6050 4650
+Wire Wire Line
+	4200 3800 3550 3800
+Wire Wire Line
+	3550 3800 3550 4950
+Wire Wire Line
+	3550 4950 2350 4950
+Connection ~ 2350 4950
+Wire Wire Line
+	2350 5650 2350 5750
+Wire Wire Line
+	2350 5750 6050 5750
+Connection ~ 6050 5750
+Wire Wire Line
+	6050 2600 6050 3700
+Wire Wire Line
+	5700 2600 5850 2600
+Wire Wire Line
+	5850 2600 6050 2600
+Wire Wire Line
+	6050 2600 7250 2600
+$Comp
+L TC1016 U?
+U 1 1 55D778C2
+P 5300 2650
+F 0 "U?" H 5450 2454 60  0000 C CNN
+F 1 "TC1016" H 5300 2850 60  0000 C CNN
+F 2 "~" H 5300 2650 60  0000 C CNN
+F 3 "~" H 5300 2650 60  0000 C CNN
+	1    5300 2650
+	-1   0    0    -1
+$EndComp
+Connection ~ 6050 2600
+Connection ~ 4600 2600
+$Comp
+L GND #PWR?
+U 1 1 55D7790B
+P 5300 3300
+F 0 "#PWR?" H 5300 3300 30  0001 C CNN
+F 1 "GND" H 5300 3230 30  0001 C CNN
+F 2 "~" H 5300 3300 60  0000 C CNN
+F 3 "~" H 5300 3300 60  0000 C CNN
+	1    5300 3300
+	1    0    0    -1
+$EndComp
+Wire Wire Line
+	5300 2900 5300 3200
+Wire Wire Line
+	5300 3200 5300 3300
+$Comp
+L C C?
+U 1 1 55D779B2
+P 5850 2950
+F 0 "C?" H 5850 3050 40  0000 L CNN
+F 1 "C" H 5856 2865 40  0000 L CNN
+F 2 "~" H 5888 2800 30  0000 C CNN
+F 3 "~" H 5850 2950 60  0000 C CNN
+	1    5850 2950
+	1    0    0    -1
+$EndComp
+$Comp
+L C C?
+U 1 1 55D779BF
+P 4800 2950
+F 0 "C?" H 4800 3050 40  0000 L CNN
+F 1 "C" H 4806 2865 40  0000 L CNN
+F 2 "~" H 4838 2800 30  0000 C CNN
+F 3 "~" H 4800 2950 60  0000 C CNN
+	1    4800 2950
+	1    0    0    -1
+$EndComp
+Wire Wire Line
+	4800 2750 4800 2600
+Connection ~ 4800 2600
+Wire Wire Line
+	5850 2750 5850 2600
+Connection ~ 5850 2600
+Wire Wire Line
+	4800 3150 4800 3200
+Wire Wire Line
+	4800 3200 5300 3200
+Wire Wire Line
+	5300 3200 5850 3200
+Connection ~ 5300 3200
+Wire Wire Line
+	5850 3200 5850 3150
+$Comp
+L POT RV?
+U 1 1 55D77A82
+P 2350 4550
+F 0 "RV?" H 2350 4450 50  0000 C CNN
+F 1 "POT" H 2350 4550 50  0000 C CNN
+F 2 "~" H 2350 4550 60  0000 C CNN
+F 3 "~" H 2350 4550 60  0000 C CNN
+	1    2350 4550
+	0    1    1    0
+$EndComp
+Wire Wire Line
+	2650 2600 2650 4550
+Wire Wire Line
+	2650 4550 2500 4550
+$Comp
+L CONN_2 P?
+U 1 1 55D77AF4
+P 7600 2700
+F 0 "P?" V 7550 2700 40  0000 C CNN
+F 1 "CONN_2" V 7650 2700 40  0000 C CNN
+F 2 "" H 7600 2700 60  0000 C CNN
+F 3 "" H 7600 2700 60  0000 C CNN
+	1    7600 2700
+	1    0    0    -1
+$EndComp
+$Comp
+L GND #PWR?
+U 1 1 55D77B0C
+P 7150 3000
+F 0 "#PWR?" H 7150 3000 30  0001 C CNN
+F 1 "GND" H 7150 2930 30  0001 C CNN
+F 2 "~" H 7150 3000 60  0000 C CNN
+F 3 "~" H 7150 3000 60  0000 C CNN
+	1    7150 3000
+	1    0    0    -1
+$EndComp
+Wire Wire Line
+	7250 2800 7150 2800
+Wire Wire Line
+	7150 2800 7150 3000
+$Comp
+L LMV358 U?
+U 2 1 55D77B6E
+P 8250 4300
+F 0 "U?" H 8200 4500 60  0000 L CNN
+F 1 "LMV358" H 8200 4050 60  0000 L CNN
+F 2 "" H 8250 4300 60  0000 C CNN
+F 3 "" H 8250 4300 60  0000 C CNN
+	2    8250 4300
+	1    0    0    -1
+$EndComp
 $EndSCHEMATC
