File: CurrentSinkOrSwim/CurrentSinkOrSwim.sch (KiCad schematic (older format))
At the start: 3 parts, among them K101 CONN_3, P101 CONN_2, P102 CONN_2

Commit message: Haciendo algunos cambios porque he tenido que cambiar de componentes y algún valor estaba mal
Parts:
- P101, P102: MFG Name MA522-500M02 -> CTB5000/2
Changed lines of the file:
@@
 Sheet 1 4
 Title ""
-Date "1 oct 2015"
+Date "5 oct 2015"
 Rev ""
 Comp ""
@@
 F 2 "" H 7600 2150 60  0000 C CNN
 F 3 "" H 7600 2150 60  0000 C CNN
-F 4 "MA522-500M02" H 7600 2150 60  0001 C CNN "MFG Name"
+F 4 "CTB5000/2" H 7600 2150 60  0001 C CNN "MFG Name"
 	1    7600 2150
 	1    0    0    -1
@@
 F 2 "" H 2650 1450 60  0000 C CNN
 F 3 "" H 2650 1450 60  0000 C CNN
-F 4 "MA522-500M02" H 2650 1450 60  0001 C CNN "MFG Name"
+F 4 "CTB5000/2" H 2650 1450 60  0001 C CNN "MFG Name"
 	1    2650 1450
 	-1   0    0    -1
