File: CurrentSinkOrSwim/CurrentControl.sch (KiCad schematic (older format))
At the start: 7 parts

Commit message: Schematic annotate
Parts:
- gave numbers to parts that had none: 7
Connections:
- net at R302.1: now also U201.7; no longer U201.1
- net at Q301.S, R303.1: now also U201.6 (-); no longer U201.2 (-)
- net at R301.1, RV301.3: now also U201.5 (+); no longer U201.3 (+)
Changed lines of the file:
@@
 Sheet 3 4
 Title ""
-Date "1 sep 2015"
+Date "6 sep 2015"
 Rev ""
 Comp ""
@@
 $EndDescr
 $Comp
-L LMV358 U?
-U 1 1 55E5E171
+L LMV358 U201
+U 2 1 55E5E171
 P 5750 3950
-F 0 "U?" H 5700 4150 60  0000 L CNN
+F 0 "U201" H 5700 4150 60  0000 L CNN
 F 1 "LMV358" H 5700 3700 60  0000 L CNN
 F 2 "" H 5750 3950 60  0000 C CNN
 F 3 "" H 5750 3950 60  0000 C CNN
-	1    5750 3950
+	2    5750 3950
 	1    0    0    -1
 $EndComp
 $Comp
-L R R?
+L R R303
 U 1 1 55E5E178
 P 8050 5200
-F 0 "R?" V 8130 5200 40  0000 C CNN
+F 0 "R303" V 8130 5200 40  0000 C CNN
 F 1 "0.1" V 8057 5201 40  0000 C CNN
 F 2 "~" V 7980 5200 30  0000 C CNN
@@
 $EndComp
 $Comp
-L MOSFET_N Q?
+L MOSFET_N Q301
 U 1 1 55E5E185
 P 7950 3950
-F 0 "Q?" H 7960 4120 60  0000 R CNN
+F 0 "Q301" H 7960 4120 60  0000 R CNN
 F 1 "BUK7575" H 7960 3800 60  0000 R CNN
 F 2 "~" H 7950 3950 60  0000 C CNN
@@
 $EndComp
 $Comp
-L R R?
+L R R301
 U 1 1 55E5E18B
 P 3400 5450
-F 0 "R?" V 3480 5450 40  0000 C CNN
+F 0 "R301" V 3480 5450 40  0000 C CNN
 F 1 "R" V 3407 5451 40  0000 C CNN
 F 2 "~" V 3330 5450 30  0000 C CNN
@@
 $EndComp
 $Comp
-L GND #PWR?
+L GND #PWR302
 U 1 1 55E5E191
 P 5650 4500
-F 0 "#PWR?" H 5650 4500 30  0001 C CNN
+F 0 "#PWR302" H 5650 4500 30  0001 C CNN
 F 1 "GND" H 5650 4430 30  0001 C CNN
 F 2 "~" H 5650 4500 60  0000 C CNN
@@
 $EndComp
 $Comp
-L POT RV?
+L POT RV301
 U 1 1 55E5E197
 P 3400 4600
-F 0 "RV?" H 3400 4500 50  0000 C CNN
+F 0 "RV301" H 3400 4500 50  0000 C CNN
 F 1 "POT" H 3400 4600 50  0000 C CNN
 F 2 "~" H 3400 4600 60  0000 C CNN
@@
 $EndComp
 $Comp
-L C C?
+L C C301
 U 1 1 55E5E19D
 P 5150 3450
-F 0 "C?" H 5150 3550 40  0000 L CNN
+F 0 "C301" H 5150 3550 40  0000 L CNN
 F 1 "C" H 5156 3365 40  0000 L CNN
 F 2 "~" H 5188 3300 30  0000 C CNN
@@
 $EndComp
 $Comp
-L GND #PWR?
+L GND #PWR301
 U 1 1 55E5E1A3
 P 5150 3700
-F 0 "#PWR?" H 5150 3700 30  0001 C CNN
+F 0 "#PWR301" H 5150 3700 30  0001 C CNN
 F 1 "GND" H 5150 3630 30  0001 C CNN
 F 2 "~" H 5150 3700 60  0000 C CNN
@@
 	8050 2950 8050 3750
 $Comp
-L R R?
+L R R302
 U 1 1 55E5E25A
 P 6650 3950
-F 0 "R?" V 6730 3950 40  0000 C CNN
+F 0 "R302" V 6730 3950 40  0000 C CNN
 F 1 "1K" V 6657 3951 40  0000 C CNN
 F 2 "~" V 6580 3950 30  0000 C CNN
