File: CurrentSinkOrSwim/PowerRegulation.sch (KiCad schematic (older format))
At the start: 6 parts

Commit message: Schematic annotate
Parts:
- gave numbers to parts that had none: 6
Changed lines of the file:
@@
 Sheet 4 4
 Title ""
-Date "1 sep 2015"
+Date "6 sep 2015"
 Rev ""
 Comp ""
@@
 $EndDescr
 $Comp
-L GND #PWR?
+L GND #PWR401
 U 1 1 55E5E55C
 P 4450 4250
-F 0 "#PWR?" H 4450 4250 30  0001 C CNN
+F 0 "#PWR401" H 4450 4250 30  0001 C CNN
 F 1 "GND" H 4450 4180 30  0001 C CNN
 F 2 "~" H 4450 4250 60  0000 C CNN
@@
 $EndComp
 $Comp
-L C C?
+L C C402
 U 1 1 55E5E562
 P 5950 4000
-F 0 "C?" H 5950 4100 40  0000 L CNN
+F 0 "C402" H 5950 4100 40  0000 L CNN
 F 1 "C" H 5956 3915 40  0000 L CNN
 F 2 "~" H 5988 3850 30  0000 C CNN
@@
 $EndComp
 $Comp
-L R R?
+L R R401
 U 1 1 55E5E568
 P 3950 3750
-F 0 "R?" V 4030 3750 40  0000 C CNN
+F 0 "R401" V 4030 3750 40  0000 C CNN
 F 1 "0" V 3957 3751 40  0000 C CNN
 F 2 "~" V 3880 3750 30  0000 C CNN
@@
 $EndComp
 $Comp
-L C C?
+L C C401
 U 1 1 55E5E56E
 P 3750 3700
-F 0 "C?" H 3750 3800 40  0000 L CNN
+F 0 "C401" H 3750 3800 40  0000 L CNN
 F 1 "C" H 3756 3615 40  0000 L CNN
 F 2 "~" H 3788 3550 30  0000 C CNN
@@
 $EndComp
 $Comp
-L LM2931ACDG U?
+L LM2931ACDG U401
 U 1 1 55E5E574
 P 4500 3150
-F 0 "U?" H 4800 2900 60  0000 C CNN
+F 0 "U401" H 4800 2900 60  0000 C CNN
 F 1 "LM2931ACDG" H 4500 3450 60  0000 C CNN
 F 2 "~" H 4450 3000 60  0000 C CNN
@@
 $EndComp
 $Comp
-L R R?
+L R R402
 U 1 1 55E5E57A
 P 5400 3300
-F 0 "R?" V 5480 3300 40  0000 C CNN
+F 0 "R402" V 5480 3300 40  0000 C CNN
 F 1 "27K" V 5407 3301 40  0000 C CNN
 F 2 "~" V 5330 3300 30  0000 C CNN
@@
 $EndComp
 $Comp
-L R R?
+L R R403
 U 1 1 55E5E580
 P 5400 3900
-F 0 "R?" V 5480 3900 40  0000 C CNN
+F 0 "R403" V 5480 3900 40  0000 C CNN
 F 1 "21.6K" V 5407 3901 40  0000 C CNN
 F 2 "~" V 5330 3900 30  0000 C CNN

Commit message: Añadiendo net list, footprints y nombres a los componentes que no lo tenían. Empezando con el layout
Changed lines of the file:
@@
 $EndDescr
 $Comp
-L GND #PWR401
+L GND #PWR07
 U 1 1 55E5E55C
 P 4450 4250
-F 0 "#PWR401" H 4450 4250 30  0001 C CNN
+F 0 "#PWR07" H 4450 4250 30  0001 C CNN
 F 1 "GND" H 4450 4180 30  0001 C CNN
 F 2 "~" H 4450 4250 60  0000 C CNN
@@
 $EndComp
 Wire Wire Line
-	5950 4200 5400 4200
-Wire Wire Line
-	5400 4200 4450 4200
-Wire Wire Line
-	4450 4200 3950 4200
-Wire Wire Line
-	3950 4200 3750 4200
+	3750 4200 5950 4200
 Wire Wire Line
 	3950 4000 3950 4200
@@
 Connection ~ 5400 4200
 Wire Wire Line
-	5400 3550 5400 3600
-Wire Wire Line
-	5400 3600 5400 3650
+	5400 3550 5400 3650
 Wire Wire Line
 	5400 3600 5050 3600
@@
 Connection ~ 5400 3600
 Wire Wire Line
-	7050 3000 5950 3000
+	4900 3000 7050 3000
 Wire Wire Line
-	5950 3000 5400 3000
-Wire Wire Line
-	5400 3000 4900 3000
-Wire Wire Line
-	4450 3550 4450 3650
-Wire Wire Line
-	4450 3650 4450 3750
-Wire Wire Line
-	4450 3750 4450 3900
-Wire Wire Line
-	4450 3900 4450 4200
-Wire Wire Line
-	4450 4200 4450 4250
+	4450 3550 4450 4250
 Connection ~ 4450 4200
 Wire Wire Line
@@
 Connection ~ 5400 3000
 Wire Wire Line
-	3650 3000 3750 3000
-Wire Wire Line
-	3750 3000 4100 3000
+	3650 3000 4100 3000
 Wire Wire Line
 	3750 3500 3750 3000
