File: CurrentSinkOrSwim/CurrentSinkOrSwim.kicad_pcb (KiCad board)
At the start: 2 copper layers, 91.7 x 60.4 mm, 23 parts, among them K101 CONN_3, P101 CONN_2, P102 CONN_2, P301 CONN_1, Q301 BUK7575, U201 LMV358, U401 LM2931ACDG

Commit message: Layout session 2
Parts:
- removed C201: C, SM0805
- R301: moved to B.Cu
- moved P101 31.9 mm to (143.6, 78.0), turned to 90 degrees
- moved RV301 20.0 mm to (127.4, 80.1), turned to 0 degrees
- moved R301 16.4 mm to (118.0, 68.7), turned to 270 degrees
- moved K101 13.2 mm to (137.7, 72.8), turned to 90 degrees
- moved P102 12.8 mm to (143.6, 66.7), turned to 90 degrees
- moved RV201 12.7 mm to (113.6, 80.1), turned to 0 degrees
- moved R302 12.6 mm to (123.6, 58.8)
- moved U201 12.1 mm to (115.7, 68.0)
- moved R202 10.8 mm to (112.3, 73.0), turned to 180 degrees
- moved R201 9.79 mm to (110.6, 62.9), turned to 180 degrees
- moved R203 8.92 mm to (109.3, 67.3), turned to 90 degrees
- moved C402 8.84 mm to (129.5, 67.0)
- moved C301 6.12 mm to (115.7, 68.7), turned to 270 degrees
- moved R303 5.30 mm to (131.9, 62.2), turned to 315 degrees
- moved U401 5.22 mm to (129.7, 70.9)
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Routing:
- net N-000009: track 0.00 -> 35.7 mm, vias 0 -> 1
- net 2.7V: track 3.14 -> 37.1 mm, vias 0 -> 3
- net N-0000014: track 0.00 -> 22.0 mm
- net GND: track 6.75 -> 27.2 mm, vias 1 -> 4
- net N-0000013: track 0.00 -> 18.1 mm, vias 0 -> 1
- net N-000007: track 0.00 -> 12.7 mm
- net N-0000011: track 0.00 -> 10.5 mm
- net N-000006: track 0.00 -> 9.39 mm
- net N-000001: track 17.3 -> 8.04 mm
- net /Current Control/FET_Gate: track 0.00 -> 8.29 mm
- net N-0000017: track 0.00 -> 5.59 mm
- net /Power Regulation/Vin: track 14.2 -> 9.38 mm, vias 1 -> 0
- net /Current Control/Current_Sink+: track 62.1 -> 66.1 mm
- net N-0000016: track 3.75 -> 3.14 mm
Other:
- board size 91.7 x 60.4 mm -> 41.7 x 47.8 mm
